File: c61/c61.kicad_pcb (KiCad board)
At the start: 2 copper layers, 21 x 37 mm, 17 parts, among them J1 1x14, J2 SFV24R-EPAPER, U1 ESP32-C61HF4, U2 TPS63900DSKR, Y1 Crystal 40MHz

Commit message: fix the pinheader footprint
Parts:
- J1: footprint Connector_PinHeader_1.00mm:PinHeader_1x14_P1.00mm_Vertical -> Connector_PinHeader_2.54mm:PinHeader_1x14_P2.54mm_Vertical
- moved J1 5.36 mm to (125.5, 93.0)
Other:
- board text added: "2026-July"
- board text added: "ESP32-C61 SIDECAR"
- board text removed: "ESP32-C61 SIDECAR 2026-Jun"
Changed lines of the file:
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@@
 		)
 	)
-	(footprint "Connector_PinHeader_1.00mm:PinHeader_1x14_P1.00mm_Vertical"
+	(footprint "Connector_PinHeader_2.54mm:PinHeader_1x14_P2.54mm_Vertical"
 		(layer "F.Cu")
-		(at 130.909938 92.922608)
-		(descr "Through hole straight pin header, 1x14, 1.00mm pitch, single row")
-		(tags "Through hole pin header THT 1x14 1.00mm single row")
+		(at 125.55 92.99)
+		(descr "Through hole straight pin header, 1x14, 2.54mm pitch, single row")
+		(tags "Through hole pin header THT 1x14 2.54mm single row")
 		(property "Reference" "J1"
-			(at -0.5 -1.16 0)
+			(at 0 -2.38 0)
 			(layer "F.SilkS")
 			(effects
 				(font
-					(size 0.3 0.3)
-					(thickness 0.075)
-					(bold yes)
+					(size 1 1)
+					(thickness 0.15)
 				)
 			)
 		)
 		(property "Value" "1x14"
-			(at 0 14.36 0)
+			(at 0 35.4 0)
 			(layer "F.Fab")
 			(effects
 				(font
-					(size 0.4 0.4)
-					(thickness 0.1)
+					(size 1 1)
+					(thickness 0.15)
 				)
 			)
@@
 		(duplicate_pad_numbers_are_jumpers no)
 		(fp_line
-			(start -0.745 -0.735)
-			(end 0 -0.735)
+			(start -1.38 -1.38)
+			(end 0 -1.38)
 			(stroke
 				(width 0.12)
@@
 		)
 		(fp_line
-			(start -0.745 0)
-			(end -0.745 -0.735)
+			(start -1.38 0)
+			(end -1.38 -1.38)
 			(stroke
 				(width 0.12)
@@
 		)
 		(fp_line
-			(start -0.745 0.735)
-			(end -0.745 13.61)
+			(start -1.38 1.27)
+			(end -1.38 34.4)
 			(stroke
 				(width 0.12)
@@
 		)
 		(fp_line
-			(start -0.745 0.735)
-			(end -0.685565 0.735)
+			(start -1.38 1.27)
+			(end 1.38 1.27)
 			(stroke
 				(width 0.12)
@@
 		)
 		(fp_line
-			(start -0.745 13.61)
-			(end -0.41003 13.61)
+			(start -1.38 34.4)
+			(end 1.38 34.4)
 			(stroke
 				(width 0.12)
@@
 		)
 		(fp_line
-			(start 0.41003 13.61)
-			(end 0.745 13.61)
+			(start 1.38 1.27)
+			(end 1.38 34.4)
 			(stroke
 				(width 0.12)
@@
 			(layer "F.SilkS")
 		)
-		(fp_line
-			(start 0.685565 0.735)
-			(end 0.745 0.735)
-			(stroke
-				(width 0.12)
-				(type solid)
-			)
-			(layer "F.SilkS")
-		)
-		(fp_line
-			(start 0.745 0.735)
-			(end 0.745 13.61)
-			(stroke
-				(width 0.12)
-				(type solid)
-			)
-			(layer "F.SilkS")
-		)
 		(fp_rect
-			(start -1.14 -1)
-			(end 1.14 14)
+			(start -1.77 -1.78)
+			(end 1.77 34.8)
 			(stroke
 				(width 0.05)
@@
 		)
 		(fp_line
-			(start -0.635 -0.1825)
-			(end -0.3175 -0.5)
+			(start -1.27 -0.635)
+			(end -0.635 -1.27)
 			(stroke
 				(width 0.1)
@@
 		)
 		(fp_line
-			(start -0.635 13.5)
-			(end -0.635 -0.1825)
+			(start -1.27 34.29)
+			(end -1.27 -0.635)
 			(stroke
 				(width 0.1)
@@
 		)
 		(fp_line
-			(start -0.3175 -0.5)
-			(end 0.635 -0.5)
+			(start -0.635 -1.27)
+			(end 1.27 -1.27)
 			(stroke
 				(width 0.1)
@@
 		)
 		(fp_line
-			(start 0.635 -0.5)
-			(end 0.635 13.5)
+			(start 1.27 -1.27)
+			(end 1.27 34.29)
 			(stroke
 				(width 0.1)
@@
 		)
 		(fp_line
-			(start 0.635 13.5)
-			(end -0.635 13.5)
+			(start 1.27 34.29)
+			(end -1.27 34.29)
 			(stroke
 				(width 0.1)
@@
 		)
 		(fp_text user "${REFERENCE}"
-			(at 0 6.5 90)
+			(at 0 16.51 90)
 			(layer "F.Fab")
 			(effects
 				(font
-					(size 0.76 0.76)
-					(thickness 0.114)
+					(size 1 1)
+					(thickness 0.15)
 				)
 			)
@@
 		(pad "1" thru_hole rect
 			(at 0 0)
-			(size 0.85 0.85)
-			(drill 0.5)
+			(size 1.7 1.7)
+			(drill 1)
 			(layers "*.Cu" "*.Mask")
 			(remove_unused_layers no)
@@
 		)
 		(pad "2" thru_hole circle
-			(at 0 1)
-			(size 0.85 0.85)
-			(drill 0.5)
+			(at 0 2.54)
+			(size 1.7 1.7)
+			(drill 1)
 			(layers "*.Cu" "*.Mask")
 			(remove_unused_layers no)
@@
 		)
 		(pad "3" thru_hole circle
-			(at 0 2)
-			(size 0.85 0.85)
-			(drill 0.5)
+			(at 0 5.08)
+			(size 1.7 1.7)
+			(drill 1)
 			(layers "*.Cu" "*.Mask")
 			(remove_unused_layers no)
@@
 		)
 		(pad "4" thru_hole circle
-			(at 0 3)
-			(size 0.85 0.85)
-			(drill 0.5)
+			(at 0 7.62)
+			(size 1.7 1.7)
+			(drill 1)
 			(layers "*.Cu" "*.Mask")
 			(remove_unused_layers no)
@@
 		)
 		(pad "5" thru_hole circle
-			(at 0 4)
-			(size 0.85 0.85)
-			(drill 0.5)
+			(at 0 10.16)
+			(size 1.7 1.7)
+			(drill 1)
 			(layers "*.Cu" "*.Mask")
 			(remove_unused_layers no)
@@
 		)
 		(pad "6" thru_hole circle
-			(at 0 5)
-			(size 0.85 0.85)
-			(drill 0.5)
+			(at 0 12.7)
+			(size 1.7 1.7)
+			(drill 1)
 			(layers "*.Cu" "*.Mask")
 			(remove_unused_layers no)
@@
 		)
 		(pad "7" thru_hole circle
-			(at 0 6)
-			(size 0.85 0.85)
-			(drill 0.5)
+			(at 0 15.24)
+			(size 1.7 1.7)
+			(drill 1)
 			(layers "*.Cu" "*.Mask")
 			(remove_unused_layers no)
@@
 		)
 		(pad "8" thru_hole circle
-			(at 0 7)
-			(size 0.85 0.85)
-			(drill 0.5)
+			(at 0 17.78)
+			(size 1.7 1.7)
+			(drill 1)
 			(layers "*.Cu" "*.Mask")
 			(remove_unused_layers no)
@@
 		)
 		(pad "9" thru_hole circle
-			(at 0 8)
-			(size 0.85 0.85)
-			(drill 0.5)
+			(at 0 20.32)
+			(size 1.7 1.7)
+			(drill 1)
 			(layers "*.Cu" "*.Mask")
 			(remove_unused_layers no)
@@
 		)
 		(pad "10" thru_hole circle
-			(at 0 9)
-			(size 0.85 0.85)
-			(drill 0.5)
+			(at 0 22.86)
+			(size 1.7 1.7)
+			(drill 1)
 			(layers "*.Cu" "*.Mask")
 			(remove_unused_layers no)
@@
 		)
 		(pad "11" thru_hole circle
-			(at 0 10)
-			(size 0.85 0.85)
-			(drill 0.5)
+			(at 0 25.4)
+			(size 1.7 1.7)
+			(drill 1)
 			(layers "*.Cu" "*.Mask")
 			(remove_unused_layers no)
@@
 		)
 		(pad "12" thru_hole circle
-			(at 0 11)
-			(size 0.85 0.85)
-			(drill 0.5)
+			(at 0 27.94)
+			(size 1.7 1.7)
+			(drill 1)
 			(layers "*.Cu" "*.Mask")
 			(remove_unused_layers no)
@@
 		)
 		(pad "13" thru_hole circle
-			(at 0 12)
-			(size 0.85 0.85)
-			(drill 0.5)
+			(at 0 30.48)
+			(size 1.7 1.7)
+			(drill 1)
 			(layers "*.Cu" "*.Mask")
 			(remove_unused_layers no)
@@
 		)
 		(pad "14" thru_hole circle
-			(at 0 13)
-			(size 0.85 0.85)
-			(drill 0.5)
+			(at 0 33.02)
+			(size 1.7 1.7)
+			(drill 1)
 			(layers "*.Cu" "*.Mask")
 			(remove_unused_layers no)
@@
 		)
 		(embedded_fonts no)
-		(model "${KICAD10_3DMODEL_DIR}/Connector_PinHeader_1.00mm.3dshapes/PinHeader_1x14_P1.00mm_Vertical.step"
+		(model "${KICAD10_3DMODEL_DIR}/Connector_PinHeader_2.54mm.3dshapes/PinHeader_1x14_P2.54mm_Vertical.step"
 			(offset
 				(xyz 0 0 0)
@@
 		(layer "Edge.Cuts")
 	)
-	(gr_text "ESP32-C61 SIDECAR 2026-Jun"
-		(at 137.572527 90.887912 0)
-		(layer "F.SilkS")
-		(effects
-			(font
-				(size 0.5 0.5)
-				(thickness 0.1)
-			)
-			(justify left bottom)
-		)
-	)
 	(gr_text "1"
 		(at 129.296491 93.207269 0)
@@
 				(thickness 0.1)
 				(bold yes)
+			)
+			(justify left bottom)
+		)
+	)
+	(gr_text "ESP32-C61 SIDECAR"
+		(at 133.502197 91.419505 0)
+		(layer "F.SilkS")
+		(effects
+			(font
+				(size 0.9 0.9)
+				(thickness 0.1)
 			)
 			(justify left bottom)
@@
 			)
 			(justify left bottom mirror)
+		)
+	)
+	(gr_text "2026-July"
+		(at 149.4 91.7 0)
+		(layer "B.SilkS")
+		(effects
+			(font
+				(size 0.8 0.8)
+				(thickness 0.1)
+			)
+			(justify left bottom mirror)

Commit message: 2.54 headers!
Parts:
- added D1: LED, LED_SMD:LED_1206_3216Metric, F.Cu at (148.2, 104.8)
- moved J1 5.37 mm to (130.8, 91.8)
Connections:
- U1 pad 36: unconnected-(U1-GPIO7-Pad36) -> Net-(D1-K)
Routing:
- net /VBUS: track 32.7 -> 23.4 mm, vias 2 -> 1
- net /HLPOW: track 22.7 -> 13.9 mm
- net Net-(D1-K): track 0.00 -> 7.84 mm, vias 0 -> 2
- net /PST2: track 28.3 -> 20.7 mm
- net /3.3V: track 36.3 -> 42.5 mm
- net /PST1: track 17.6 -> 13.5 mm
- net GND: track 104.9 -> 101.6 mm, vias 17 -> 18
- net /A34: track 15.2 -> 12.8 mm
- net Net-(J1-Pin_4): track 16.0 -> 14.0 mm
- net Net-(J1-Pin_3): track 33.0 -> 33.8 mm
- net Net-(C1-Pad2): track 6.57 -> 5.81 mm
- net /A12: track 15.3 -> 16.0 mm
Other:
- board text removed: "1"
