File: c61/c61.kicad_pcb (KiCad board)
At the start: 2 copper layers, 21 x 37 mm, 18 parts, among them J1 1x14, J2 SFV24R-EPAPER, U1 ESP32-C61HF4, U2 TPS63900DSKR, Y1 Crystal 40MHz

Commit message: 12pF for 40mhz crystal
Parts:
- removed J2: SFV24R-EPAPER, somethingfootprints:SFV24R3STBE1HLF
- C1, C2: value 22nF -> 12pF

Commit message: c61 improvements
Parts:
- added C5: 22uF, Capacitor_SMD:C_0805_2012Metric_Pad1.18x1.45mm_HandSolder, F.Cu at (136.8, 119.8)
- added C7: 10uF, Capacitor_SMD:C_0805_2012Metric_Pad1.18x1.45mm_HandSolder, F.Cu at (136.7, 114.8)
- added R9: 200R, Resistor_SMD:R_0603_1608Metric_Pad0.98x0.95mm_HandSolder, F.Cu at (148.1, 99.7)
- C4: footprint Capacitor_SMD:C_0603_1608Metric_Pad1.08x0.95mm_HandSolder -> Capacitor_SMD:C_0805_2012Metric_Pad1.18x1.45mm_HandSolder
- R1, R2: footprint Resistor_SMD:R_0603_1608Metric_Pad0.98x0.95mm_HandSolder -> Resistor_SMD:R_0805_2012Metric_Pad1.20x1.40mm_HandSolder
- Y1: footprint Crystal:Crystal_SMD_3225-4Pin_3.2x2.5mm_HandSoldering -> Crystal:Crystal_SMD_3225-4Pin_3.2x2.5mm
- moved D1 9.24 mm to (148.2, 95.6)
- moved C2 4.89 mm to (143.2, 98.6), turned to 90 degrees
- moved L2 4.11 mm to (143.9, 118.2)
- moved Y1 3.59 mm to (140.1, 98.6)
- moved C1 2.71 mm to (137.1, 98.7)
- moved C4 2.67 mm to (136.5, 104.9)
- moved L1 2.11 mm to (140.4, 102.7)
- moved U2 1.87 mm to (141.1, 118.1)
- moved R8 1.68 mm to (143.4, 102.7)
- moved R2 0.68 mm to (136.8, 118.2)
- moved R1 0.17 mm to (136.8, 116.7)
Connections:
- J1 pad 12: /HLPOW -> /VBUS
- J1 pad 13: unconnected-(J1-Pin_13-Pad13) -> /HLPOW
- J1 pad 14: unconnected-(J1-Pin_14-Pad14) -> /3.3V
- J1 pad 6: /VBUS -> /D+
- J1 pad 7: /3.3V -> /D-
- U1 pad 28: unconnected-(U1-USB_D--Pad28) -> /D-
- U1 pad 29: unconnected-(U1-USB_D+-Pad29) -> /D+
- U1 pad 36: Net-(D1-K) -> Net-(U1-GPIO7)
Routing:
- net GND: track 101.6 -> 6.05 mm, vias 18 -> 72
- net /3.3V: track 42.5 -> 15.5 mm
- net /D-: track 0.00 -> 19.6 mm, vias 0 -> 1
- net /D+: track 0.00 -> 18.5 mm, vias 0 -> 1
- net Net-(J1-Pin_4): track 14.0 -> 24.3 mm, vias 2 -> 0
- net Net-(U1-GPIO7): track 0.00 -> 9.44 mm, vias 0 -> 2
- net /ANT: track 25.4 -> 16.4 mm, vias 4 -> 2
- net Net-(J1-Pin_3): track 33.8 -> 27.0 mm
- net Net-(J1-Pin_2): track 33.3 -> 26.5 mm
- net Net-(U1-XTAL_N): track 17.4 -> 11.3 mm
- net Net-(D1-K): track 7.84 -> 1.86 mm, vias 2 -> 0
- net Net-(J1-Pin_1): track 33.1 -> 28.0 mm
- net /VBUS: track 23.4 -> 20.9 mm, vias 1 -> 0
- net Net-(U2-LX1): track 3.97 -> 1.75 mm
- net Net-(U2-LX2): track 3.99 -> 1.81 mm
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- added copper zone on F.Cu, net GND
Other:
- board text added: "2026-Aug"
- board text added: "D+"
- board text added: "D-"
- board text removed: "2026-July"
